File: PCB/PCB.kicad_pcb (KiCad board)
At the start: 2 copper layers, 47 parts, among them J4 Conn_01x15_Pin, J5 Conn_01x15_Pin, U1 AMS1117-3.3, U3 YZA-056-4.3, U4 YZA-056-4.3, U5 ESP32-S3, X1 TXM40M0004322HBCEO00T

Commit message: restart again
Parts:
- removed the C1 at (103.6, 155.8)
- removed the C1 at (91.5, 153.3)
- removed the C18 at (106.4, 135.2)
- removed the C18 at (91.5, 158.7)
- removed C23, C24: CL31A106KBHNNNE, easyeda2kicad:C1206
- removed the C6 at (94.8, 153.0)
- removed the C6 at (83.8, 137.5)
- removed the C7 at (104.8, 137.2)
- removed the C7 at (94.8, 154.9)
- removed the C9 at (109.0, 132.2)
- removed the C9 at (94.8, 156.8)
- added C1: CL10A106MA8NRNC, easyeda2kicad:C0603, F.Cu at (93.8, 153.3)
- added C18: CL10A106MA8NRNC, easyeda2kicad:C0603, F.Cu at (92.2, 142.2)
- added C6: 0201CG1R5C500NT, easyeda2kicad:C0201, F.Cu at (133.4, 168.0)
- added C7: 0201CG1R5C500NT, easyeda2kicad:C0201, F.Cu at (133.4, 169.9)
- added C9: 0201CG1R5C500NT, easyeda2kicad:C0201, F.Cu at (133.4, 171.9)
- moved J5 49.4 mm to (107.8, 173.1), turned to 180 degrees
- moved J4 49.2 mm to (84.2, 173.1), turned to 180 degrees
- moved C12 41.5 mm to (133.4, 173.8)
- moved R2 38.1 mm to (87.8, 164.8), turned to -90 degrees
- moved L4 37.8 mm to (116.5, 173.7)
- moved C8 34.6 mm to (100.5, 165.5), turned to 90 degrees
- moved L2 34.3 mm to (116.5, 171.8), turned to 0 degrees
- moved L1 33.0 mm to (116.5, 169.9), turned to 0 degrees
- moved C14 32.6 mm to (116.7, 165.7), turned to 0 degrees
- moved C13 27.6 mm to (92.2, 143.8), turned to 0 degrees
- moved C4 26.1 mm to (116.7, 159.2)
- moved C16 26.1 mm to (92.3, 145.2), turned to 0 degrees
- moved D1 25.2 mm to (132.7, 138.8)
- moved X1 25.2 mm to (130.6, 164.6), turned to 0 degrees
- moved U5 24.4 mm to (96.2, 162.1)
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Routing:
- net GND: track 89.7 -> 1.52 mm, vias 20 -> 0
- net /CHIP_EN: track 34.5 -> 89.0 mm, vias 4 -> 0
- net +3V3: track 83.2 -> 133.0 mm, vias 8 -> 0
- net Net-(U5-XTAL_P): track 40.7 -> 0.00 mm, vias 2 -> 0
- net GPIO12: track 35.1 -> 0.00 mm, vias 1 -> 0
- net GPIO17: track 20.8 -> 53.8 mm, vias 1 -> 2
- net Net-(X1-OSC1): track 30.1 -> 0.00 mm, vias 4 -> 0
- net GPIO11: track 44.8 -> 15.6 mm
- net GPIO10: track 48.9 -> 19.6 mm
- net Net-(U5-XTAL_N): track 21.9 -> 0.00 mm, vias 3 -> 0
- net VSYS: track 52.7 -> 74.3 mm, vias 4 -> 0
- net GPIO35: track 19.9 -> 0.00 mm
- net GPIO18: track 21.4 -> 40.5 mm, vias 1 -> 2
- net GPIO37: track 17.9 -> 0.00 mm
- net GPIO36: track 17.8 -> 0.00 mm
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
Commit message: final commit i hope
Parts:
- removed C22: CL31A106KBHNNNE, easyeda2kicad:C1206
- added C19: CL10A106MA8NRNC, easyeda2kicad:C0603, F.Cu at (94.0, 137.0)
- added G***: LOGO, LOGO, B.Cu at (92.8, 163.8)
- added G***: LOGO, LOGO, B.Cu at (85.8, 166.8)
- moved C12 62.4 mm to (82.5, 137.8)
- moved C9 60.6 mm to (84.0, 136.8)
- moved C6 59.0 mm to (84.0, 135.8)
- moved C7 53.1 mm to (83.5, 151.8), turned to 90 degrees
- moved D1 50.3 mm to (82.5, 135.8)
- moved L4 50.2 mm to (82.5, 136.8), turned to 180 degrees
- moved X1 49.0 mm to (89.0, 138.8)
- moved L3 43.1 mm to (87.5, 146.8), turned to 90 degrees
- moved C14 40.5 mm to (89.2, 136.0), turned to 180 degrees
- moved R1 39.0 mm to (91.0, 167.0), turned to 180 degrees
- moved L1 38.1 mm to (82.5, 152.8), turned to 90 degrees
- moved L2 37.8 mm to (85.2, 150.5), turned to 90 degrees
- moved C15 37.4 mm to (87.5, 144.5), turned to -90 degrees
- moved C4 33.4 mm to (84.2, 151.3), turned to 90 degrees
- moved C11 33.1 mm to (91.5, 165.8)
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Connections:
- J4 pad 1: /VIN -> GPIO14
- J4 pad 12: GPIO14 -> /VIN
- J4 pad 13: GPIO18 -> /U0TXD
- J4 pad 14: GPIO17 -> /U0RXD
- J4 pad 2: /U0TXD -> GPIO18
- J4 pad 3: /U0RXD -> GPIO17
- J5 pad 10: GPIO38 -> GPIO35
- J5 pad 11: GPIO37 -> GPIO36
- J5 pad 12: GPIO36 -> GPIO37
- J5 pad 13: GPIO35 -> GPIO38
- J5 pad 14: GPIO34 -> GPIO39
- J5 pad 15: GPIO33 -> GPIO40
- J5 pad 3: GPIO13 -> GPIO9
- J5 pad 4: GPIO12 -> GPIO10
- J5 pad 6: GPIO10 -> GPIO12
- J5 pad 7: GPIO9 -> GPIO13
- J5 pad 8: GPIO40 -> GPIO33
- J5 pad 9: GPIO39 -> GPIO34
- U5 pad : (no net) -> GND
Routing:
- net GND: track 1.52 -> 122.2 mm, vias 0 -> 34
- net /CHIP_EN: track 89.0 -> 45.9 mm, vias 0 -> 3
- net GPIO17: track 53.8 -> 22.2 mm, vias 2 -> 1
- net GPIO33: track 30.6 -> 9.73 mm, vias 2 -> 1
- net Net-(C6-Pad1): track 0.00 -> 19.9 mm, vias 0 -> 2
- net GPIO12: track 0.00 -> 19.8 mm, vias 0 -> 1
- net Net-(U5-XTAL_N): track 0.00 -> 18.0 mm, vias 0 -> 2
- net GPIO9: track 25.0 -> 42.0 mm, vias 2 -> 1
- net GPIO18: track 40.5 -> 24.3 mm, vias 2 -> 1
- net GPIO34: track 25.3 -> 10.5 mm, vias 2 -> 1
- net GPIO0: track 66.4 -> 53.7 mm, vias 2 -> 4
- net GPIO37: track 0.00 -> 11.7 mm, vias 0 -> 1
- net +3V3: track 133.0 -> 121.4 mm
- net USB_DP: track 7.12 -> 18.1 mm
- net GPIO13: track 31.9 -> 21.0 mm, vias 2 -> 1
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Other:
- board outline added: 28 x 48.2 mm
- board text added: "penguin32"

Commit message: final commit
Parts:
- removed C12, C6, C7, C9: 0201CG1R5C500NT, easyeda2kicad:C0201
- removed D1: PESD4V0Z1BSFYL, easyeda2kicad:DSN0603-2_L0.7-W0.3-P0.40-BI
- added C20: GJM1555C1H1R5BB01D, easyeda2kicad:C0402, F.Cu at (81.7, 136.9)
- added C21: GJM1555C1H1R5BB01D, easyeda2kicad:C0402, F.Cu at (79.5, 135.0)
- added C22: GJM1555C1H1R5BB01D, easyeda2kicad:C0402, F.Cu at (83.8, 136.0)
- added C23: GJM1555C1H1R5BB01D, easyeda2kicad:C0402, F.Cu at (81.6, 153.8)
- added U2: H5VU10BB, easyeda2kicad:DFN1006-2L-BI, F.Cu at (82.4, 135.2)
- L1, L2, L4: value SDCL0603Q2N0ST02 -> SDCL1005C2N0STDF; footprint easyeda2kicad:L0201 -> easyeda2kicad:L0402
- moved L2 15.2 mm to (79.2, 136.6)
- moved L1 3.59 mm to (85.1, 150.2)
- moved L4 2.03 mm to (80.8, 135.8), turned to 0 degrees
Connections:
- L1 pad 1: Net-(U5-LNA_IN) -> Net-(C4-Pad1)
- L1 pad 2: Net-(C6-Pad1) -> +3V3
- L2 pad 1: Net-(C4-Pad1) -> Net-(U5-LNA_IN)
- L2 pad 2: +3V3 -> Net-(C21-Pad1)
- L4 pad 1: Net-(C6-Pad1) -> Net-(C21-Pad1)
- U5 pad : GND -> (no net)
Routing:
- net +3V3: track 121.4 -> 61.1 mm, vias 0 -> 3
- net Net-(U5-LNA_IN): track 9.92 -> 34.2 mm, vias 2 -> 4
- net Net-(C6-Pad1): track 19.9 -> 0.00 mm, vias 2 -> 0
- net Net-(C21-Pad1): track 0.00 -> 8.50 mm, vias 0 -> 2
- net GND: track 122.2 -> 117.0 mm, vias 34 -> 45
- net GPIO0: track 53.7 -> 55.2 mm
- added copper zone on F.Cu, net +3V3
